Commit message: Fix beta urdf

File: tc_orne_beta/models/urdf/orne_beta.urdf (robot description, URDF)
Before this commit: robot orne_beta, 15 links, 14 joints
Links:
- removed link front_camera
- added link d435_link, mass 0.4; collision box size=0.02 0.12 0.02; visual box size=0.02 0.12 0.02
Joints:
- removed joint front_camera_joint
- added joint d435_link_joint: type fixed, parent computer_unit_link, child d435_link, origin xyz=0.24 0.0  0.05 rpy=3.14 0.35 0.0
- joint rear_laser_scan_joint: origin xyz=-0.2 0.0 -0.38 rpy=0.0 0.0 1.57 -> xyz=-0.2 0.0 -0.38 rpy=0.0 0.0 3.15
